File: CESP.sch (KiCad schematic (older format))
At the start: 5 parts

Commit message: second commit
Parts:
- removed U?: LTC1594CS, TSSOP14, symbol LTC1594CS
- removed U?: TL074, TSSOP14, symbol TL074
- removed U? (x3): TL074, symbol TL074
- added C1, C2, C3: C, ~, symbol C
- added R1, R2, R3: R, ~, symbol R
Connections:
- net labels added: +5V, GND
- wire segments 0 -> 10
Other:
- note removed: "NOTE: THIS IS JUST A TEST BOARD\nREMOVE ALL COMPONENTS AND CREATE YOUR OWN\nINCLUDE SCHEMATIC HOOKUPS/NETLIST"
Changed lines of the file:
@@
-EESchema Schematic File Version 2  date 1/24/2014 12:04:40 AM
+EESchema Schematic File Version 2
 LIBS:power
 LIBS:device
@@
 Sheet 1 1
 Title ""
-Date "24 jan 2014"
+Date "26 jan 2014"
 Rev ""
 Comp ""
@@
 $EndDescr
 $Comp
-L LTC1594CS U?
-U 1 1 52E1F38F
-P 3750 3300
-F 0 "U?" H 3750 3950 60  0000 C CNN
-F 1 "LTC1594CS" H 3750 2650 60  0000 C CNN
-F 2 "TSSOP14" H 3750 3300 60  0000 C CNN
-F 3 "" H 3750 3300 60  0000 C CNN
-	1    3750 3300
+L R R1
+U 1 1 52E56104
+P 2950 1650
+F 0 "R1" V 3030 1650 40  0000 C CNN
+F 1 "R" V 2957 1651 40  0000 C CNN
+F 2 "~" V 2880 1650 30  0000 C CNN
+F 3 "~" H 2950 1650 30  0000 C CNN
+	1    2950 1650
+	0    -1   -1   0
+$EndComp
+$Comp
+L R R2
+U 1 1 52E56113
+P 3650 1650
+F 0 "R2" V 3730 1650 40  0000 C CNN
+F 1 "R" V 3657 1651 40  0000 C CNN
+F 2 "~" V 3580 1650 30  0000 C CNN
+F 3 "~" H 3650 1650 30  0000 C CNN
+	1    3650 1650
+	0    -1   -1   0
+$EndComp
+$Comp
+L R R3
+U 1 1 52E56122
+P 4350 1650
+F 0 "R3" V 4430 1650 40  0000 C CNN
+F 1 "R" V 4357 1651 40  0000 C CNN
+F 2 "~" V 4280 1650 30  0000 C CNN
+F 3 "~" H 4350 1650 30  0000 C CNN
+	1    4350 1650
+	0    1    1    0
+$EndComp
+$Comp
+L C C1
+U 1 1 52E56189
+P 2900 2000
+F 0 "C1" H 2900 2100 40  0000 L CNN
+F 1 "C" H 2906 1915 40  0000 L CNN
+F 2 "~" H 2938 1850 30  0000 C CNN
+F 3 "~" H 2900 2000 60  0000 C CNN
+	1    2900 2000
+	0    -1   -1   0
+$EndComp
+$Comp
+L C C2
+U 1 1 52E56198
+P 3600 2000
+F 0 "C2" H 3600 2100 40  0000 L CNN
+F 1 "C" H 3606 1915 40  0000 L CNN
+F 2 "~" H 3638 1850 30  0000 C CNN
+F 3 "~" H 3600 2000 60  0000 C CNN
+	1    3600 2000
+	0    -1   -1   0
+$EndComp
+$Comp
+L C C3
+U 1 1 52E561C6
+P 4300 2000
+F 0 "C3" H 4300 2100 40  0000 L CNN
+F 1 "C" H 4306 1915 40  0000 L CNN
+F 2 "~" H 4338 1850 30  0000 C CNN
+F 3 "~" H 4300 2000 60  0000 C CNN
+	1    4300 2000
+	0    -1   -1   0
+$EndComp
+$Comp
+L +5V #PWR1
+U 1 1 52E5626F
+P 2350 1300
+F 0 "#PWR1" H 2350 1390 20  0001 C CNN
+F 1 "+5V" H 2350 1390 30  0000 C CNN
+F 2 "" H 2350 1300 60  0000 C CNN
+F 3 "" H 2350 1300 60  0000 C CNN
+	1    2350 1300
 	1    0    0    -1
 $EndComp
+Wire Wire Line
+	3200 1650 3400 1650
+Wire Wire Line
+	3900 1650 4100 1650
+Wire Wire Line
+	3100 2000 3400 2000
+Wire Wire Line
+	3800 2000 4100 2000
+Wire Wire Line
+	2350 1300 2350 2150
+Wire Wire Line
+	2700 2000 2350 2000
+Connection ~ 2350 2000
+Wire Wire Line
+	2350 1650 2700 1650
+Connection ~ 2350 1650
 $Comp
-L TL074 U?
-U 1 1 52E1F3CD
-P 7150 2150
-F 0 "U?" H 7200 2350 60  0000 C CNN
-F 1 "TL074" H 7300 1950 50  0000 C CNN
-F 2 "TSSOP14" H 7150 2150 60  0000 C CNN
-F 3 "" H 7150 2150 60  0000 C CNN
-	1    7150 2150
+L GND #PWR2
+U 1 1 52E562CA
+P 4750 2400
+F 0 "#PWR2" H 4750 2400 30  0001 C CNN
+F 1 "GND" H 4750 2330 30  0001 C CNN
+F 2 "" H 4750 2400 60  0000 C CNN
+F 3 "" H 4750 2400 60  0000 C CNN
+	1    4750 2400
 	1    0    0    -1
 $EndComp
-$Comp
-L TL074 U?
-U 2 1 52E1F3DA
-P 7200 3500
-F 0 "U?" H 7250 3700 60  0000 C CNN
-F 1 "TL074" H 7350 3300 50  0000 C CNN
-F 2 "" H 7200 3500 60  0000 C CNN
-F 3 "" H 7200 3500 60  0000 C CNN
-	2    7200 3500
-	1    0    0    -1
-$EndComp
-$Comp
-L TL074 U?
-U 1 1 52E1F3E5
-P 8600 3500
-F 0 "U?" H 8650 3700 60  0000 C CNN
-F 1 "TL074" H 8750 3300 50  0000 C CNN
-F 2 "" H 8600 3500 60  0000 C CNN
-F 3 "" H 8600 3500 60  0000 C CNN
-	1    8600 3500
-	1    0    0    -1
-$EndComp
-$Comp
-L TL074 U?
-U 1 1 52E1F3EB
-P 8550 2100
-F 0 "U?" H 8600 2300 60  0000 C CNN
-F 1 "TL074" H 8700 1900 50  0000 C CNN
-F 2 "" H 8550 2100 60  0000 C CNN
-F 3 "" H 8550 2100 60  0000 C CNN
-	1    8550 2100
-	1    0    0    -1
-$EndComp
-Text Notes 4450 4650 0    80   ~ 0
-NOTE: THIS IS JUST A TEST BOARD\nREMOVE ALL COMPONENTS AND CREATE YOUR OWN\nINCLUDE SCHEMATIC HOOKUPS/NETLIST
+Wire Wire Line
+	4600 1650 4750 1650
+Wire Wire Line
+	4750 1650 4750 2400
+Wire Wire Line
+	4500 2000 4750 2000
+Connection ~ 4750 2000
 $EndSCHEMATC
